Commit message: 实现moveit控制仿真以及实际机器人

File: src/arm_description/urdf/arm_description.xacro (robot description, xacro)
@@ -30,24 +30,24 @@
     <xacro:property name="servo_0_height" value="0.0350" />
     <xacro:property name="servo_0_mass" value="0.05" />
-    <xacro:property name="servo_0_min_pos" value="-${pi}" />
-    <xacro:property name="servo_0_max_pos" value="${pi}" />
+    <xacro:property name="servo_0_min_pos" value="-${pi/4}" />
+    <xacro:property name="servo_0_max_pos" value="${pi/4}" />
     <xacro:property name="servo_1_length" value="0.0442" />
     <xacro:property name="servo_1_width" value="0.020" />
     <xacro:property name="servo_1_height" value="0.03715" />
     <xacro:property name="servo_1_mass" value="0.05" />
-    <xacro:property name="servo_1_min_pos" value="-${pi/2}" />
-    <xacro:property name="servo_1_max_pos" value="${pi/2}" />
+    <xacro:property name="servo_1_min_pos" value="-${pi/4}" />
+    <xacro:property name="servo_1_max_pos" value="${0}" />
     <xacro:property name="servo_2_length" value="0.0556" />
     <xacro:property name="servo_2_width" value="0.020" />
     <xacro:property name="servo_2_height" value="0.064" />
     <xacro:property name="servo_2_mass" value="0.08" />
-    <xacro:property name="servo_2_min_pos" value="-${pi/2}" />
-    <xacro:property name="servo_2_max_pos" value="${pi/2}" />
+    <xacro:property name="servo_2_min_pos" value="-${pi/4}" />
+    <xacro:property name="servo_2_max_pos" value="${0}" />
     <xacro:property name="servo_3_length" value="0.0516" />
     <xacro:property name="servo_3_width" value="0.020" />
     <xacro:property name="servo_3_height" value="${joint_connect_radius + 0.064}" />
     <xacro:property name="servo_3_mass" value="0.08" />
-    <xacro:property name="servo_3_min_pos" value="-${pi/2}" />
-    <xacro:property name="servo_3_max_pos" value="${pi/2}" />
+    <xacro:property name="servo_3_min_pos" value="-${pi}" />
+    <xacro:property name="servo_3_max_pos" value="${pi}" />
     <xacro:property name="servo_4_length" value="0.0442" />
     <xacro:property name="servo_4_width" value="0.020" />
@@ -339,5 +339,5 @@
             <plugin filename="libgz_ros2_control-system.so"
                 name="gz_ros2_control::GazeboSimROS2ControlPlugin">
-                <parameters>$(find arm_description)/config/arm_controllers.yaml</parameters>
+                <parameters>$(find arm_description)/config/arm_controllers_sim.yaml</parameters>
             </plugin>
         </gazebo>

File: src/arm_description/urdf/ros2_control.xacro (robot description, xacro)
@@ -15,4 +15,5 @@
                     <param name="write_velocity_tolerance">0.001</param>
                     <param name="write_acceleration_tolerance">0.001</param>
+                    <param name="update_rate">10</param>
                 </xacro:unless>
             </hardware>

Commit message: 增加mock测试

File: src/arm_description/urdf/arm_description.xacro (robot description, xacro)
@@ -2,4 +2,5 @@
 <robot xmlns:xacro="http://ros.org/wiki/xacro" name="base">
     <xacro:arg name="use_sim" default="false" />
+    <xacro:arg name="use_mock_hardware" default="false" />
     <xacro:macro name="box_inertial" params="mass x y z">
         <inertial>
@@ -297,5 +298,8 @@
     </joint>
     <xacro:include filename="$(find arm_description)/urdf/ros2_control.xacro" />
-    <xacro:arm_ros2_control name="SixAxisServoArm" use_sim="$(arg use_sim)" />
+    <xacro:arm_ros2_control
+        name="SixAxisServoArm"
+        use_sim="$(arg use_sim)"
+        use_mock_hardware="$(arg use_mock_hardware)" />
     <xacro:if value="$(arg use_sim)">
         <!-- 仿真时禁用重力，避免控制器激活前机械臂倒塌 -->

File: src/arm_description/urdf/ros2_control.xacro (robot description, xacro)
@@ -1,10 +1,15 @@
 <?xml version="1.0"?>
 <robot xmlns:xacro="http://www.ros.org/wiki/xacro">
-    <xacro:macro name="arm_ros2_control" params="name use_sim:=false">
+    <xacro:macro name="arm_ros2_control" params="name use_sim:=false use_mock_hardware:=false">
         <ros2_control name="SixAxisServoArm" type="system">
             <hardware>
                 <xacro:if value="${use_sim}">
-                    <plugin>gz_ros2_control/GazeboSimSystem</plugin>
-                    <param name="position_proportional_gain">50.0</param>
+                    <xacro:if value="${use_mock_hardware}">
+                        <plugin>mock_components/GenericSystem</plugin>
+                    </xacro:if>
+                    <xacro:unless value="${use_mock_hardware}">
+                        <plugin>gz_ros2_control/GazeboSimSystem</plugin>
+                        <param name="position_proportional_gain">50.0</param>
+                    </xacro:unless>
                 </xacro:if>
                 <xacro:unless value="${use_sim}">
